File: reference-design/reference-design.kicad_pcb (KiCad board)
At the start: 2 copper layers, 104 x 83.9 mm, 30 parts

Commit message: create zones for interference testing
Parts:
- H1, H10, H13, H14, H2, H5, H6, H9: footprint AH49FNTR_G1:SC59_DIO_KeyswitchOutline -> AH49FNTR_G1:SC59_DIO_KeyswitchOutline_NoRuleArea
- H16: footprint AH49FNTR_G1:SC59_DIO_KeyswitchOutline_NoRuleArea -> AH49FNTR_G1:SC59_DIO_KeyswitchOutline
Routing:
- net col2: track 148.7 -> 149.5 mm
- net row1: track 139.5 -> 140.2 mm
Other:
- board text added: "ParaKeyt Reference r0.8 UMass ECE SDP26 Team 32 Bennett Gilig, Raffi Belorian, Rikhav Shah, Shlok Raval, Theo Krueger. THIS SIDE FACE DOWN"
- board text added: "Some areas intentionally have a filled/unfilled zone for interference tests"
- board text removed: "ParaKeyt Reference r0.7 UMass ECE SDP26 Team 32 Bennett Gilig, Raffi Belorian, Rikhav Shah, Shlok Raval, Theo Krueger. THIS SIDE FACE DOWN"
- board text removed: "^ This (H16) intentionally has a filled zone for interference tests"
